File: ZoneECU.kicad_sch (KiCad schematic)
At the start: 17 parts, among them J1 5007620481, J2 Conn_02x03_Odd_Even, SW1 SW_Push, U1 STM32F103RBTx, Y1 Crystal

Commit message: Swapped USART1 RX/TX, added pull ups for USART lines
Connections:
- net USART1_RX: now also U1.43 (PA10); no longer U1.42 (PA9)
- net USART1_TX: now also U1.42 (PA9); no longer U1.43 (PA10)
Changed lines of the file:
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@@
 		)
 	)
-	(label "USART1_RX"
+	(label "USART1_TX"
 		(at 168.91 72.39 180)
 		(effects
@@
 		)
 	)
-	(label "USART1_TX"
+	(label "USART1_RX"
 		(at 168.91 74.93 180)
 		(effects

Commit message: Add serial resistors on input pins
Connections:
- net IN1: no longer U1.14 (PA0)
- net IN2: no longer U1.15 (PA1)
- net IN3: no longer U1.16 (PA2)
- net IN4: no longer U1.17 (PA3)
- net IN5: no longer U1.20 (PA4)
- net IN6: no longer U1.21 (PA5)
- net IN7: no longer U1.22 (PA6)
- net IN8: no longer U1.23 (PA7)
- new net IN_MCU1: U1.14 (PA0)
- new net IN_MCU2: U1.15 (PA1)
- new net IN_MCU3: U1.16 (PA2)
- new net IN_MCU4: U1.17 (PA3)
- new net IN_MCU5: U1.20 (PA4)
- new net IN_MCU6: U1.21 (PA5)
- new net IN_MCU7: U1.22 (PA6)
- new net IN_MCU8: U1.23 (PA7)
Other:
- sheet INPUTS ports: added IN_MCU_1, IN_MCU_2, IN_MCU_3, IN_MCU_4, IN_MCU_5, IN_MCU_6, IN_MCU_7, IN_MCU_8; removed none
Changed lines of the file:
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@@
 	(wire
 		(pts
+			(xy 62.23 182.88) (xy 72.39 182.88)
+		)
+		(stroke
+			(width 0)
+			(type default)
+		)
+	)
+	(wire
+		(pts
 			(xy 38.1 26.67) (xy 46.99 26.67)
 		)
@@
 	(wire
 		(pts
+			(xy 62.23 187.96) (xy 72.39 187.96)
+		)
+		(stroke
+			(width 0)
+			(type default)
+		)
+	)
+	(wire
+		(pts
+			(xy 62.23 190.5) (xy 72.39 190.5)
+		)
+		(stroke
+			(width 0)
+			(type default)
+		)
+	)
+	(wire
+		(pts
 			(xy 238.76 121.92) (xy 250.19 121.92)
 		)
@@
 	(wire
 		(pts
+			(xy 62.23 185.42) (xy 72.39 185.42)
+		)
+		(stroke
+			(width 0)
+			(type default)
+		)
+	)
+	(wire
+		(pts
+			(xy 62.23 180.34) (xy 72.39 180.34)
+		)
+		(stroke
+			(width 0)
+			(type default)
+		)
+	)
+	(wire
+		(pts
 			(xy 237.49 96.52) (xy 250.19 96.52)
 		)
@@
 	(wire
 		(pts
+			(xy 62.23 177.8) (xy 72.39 177.8)
+		)
+		(stroke
+			(width 0)
+			(type default)
+		)
+	)
+	(wire
+		(pts
 			(xy 187.96 60.96) (xy 198.12 60.96)
 		)
@@
 	(wire
 		(pts
+			(xy 62.23 172.72) (xy 72.39 172.72)
+		)
+		(stroke
+			(width 0)
+			(type default)
+		)
+	)
+	(wire
+		(pts
 			(xy 44.45 54.61) (xy 55.88 54.61)
 		)
@@
 	(wire
 		(pts
+			(xy 62.23 175.26) (xy 72.39 175.26)
+		)
+		(stroke
+			(width 0)
+			(type default)
+		)
+	)
+	(wire
+		(pts
 			(xy 133.35 20.32) (xy 133.35 21.59)
 		)
@@
 		)
 	)
-	(label "IN1"
+	(label "IN_MCU1"
 		(at 163.83 49.53 180)
 		(effects
@@
 		)
 	)
+	(label "IN_MCU5"
+		(at 72.39 182.88 180)
+		(effects
+			(font
+				(size 1.27 1.27)
+			)
+			(justify right bottom)
+		)
+	)
 	(label "HS1_VOUT3"
 		(at 72.39 144.78 180)
@@
 		)
 	)
+	(label "IN_MCU3"
+		(at 72.39 177.8 180)
+		(effects
+			(font
+				(size 1.27 1.27)
+			)
+			(justify right bottom)
+		)
+	)
 	(label "HS2_EN2"
 		(at 106.68 105.41 0)
@@
 		)
 	)
+	(label "IN_MCU4"
+		(at 72.39 180.34 180)
+		(effects
+			(font
+				(size 1.27 1.27)
+			)
+			(justify right bottom)
+		)
+	)
 	(label "CAN_EN"
 		(at 168.91 82.55 180)
@@
 		)
 	)
+	(label "IN_MCU6"
+		(at 72.39 185.42 180)
+		(effects
+			(font
+				(size 1.27 1.27)
+			)
+			(justify right bottom)
+		)
+	)
 	(label "3V3"
 		(at 218.44 54.61 0)
@@
 		)
 	)
-	(label "IN6"
+	(label "IN_MCU6"
 		(at 163.83 62.23 180)
 		(effects
@@
 		)
 	)
-	(label "IN4"
+	(label "IN_MCU4"
 		(at 163.83 57.15 180)
 		(effects
@@
 		)
 	)
-	(label "IN2"
+	(label "IN_MCU2"
 		(at 163.83 52.07 180)
 		(effects
@@
 		)
 	)
-	(label "IN7"
+	(label "IN_MCU7"
 		(at 163.83 64.77 180)
 		(effects
@@
 		)
 	)
-	(label "IN5"
+	(label "IN_MCU5"
 		(at 163.83 59.69 180)
 		(effects
@@
 		)
 	)
+	(label "IN_MCU2"
+		(at 72.39 175.26 180)
+		(effects
+			(font
+				(size 1.27 1.27)
+			)
+			(justify right bottom)
+		)
+	)
 	(label "HS2_SEL0"
 		(at 105.41 74.93 0)
@@
 		)
 	)
+	(label "IN_MCU8"
+		(at 72.39 190.5 180)
+		(effects
+			(font
+				(size 1.27 1.27)
+			)
+			(justify right bottom)
+		)
+	)
 	(label "HS1_EN3"
 		(at 24.13 144.78 0)
@@
 		)
 	)
+	(label "IN_MCU1"
+		(at 72.39 172.72 180)
+		(effects
+			(font
+				(size 1.27 1.27)
+			)
+			(justify right bottom)
+		)
+	)
 	(label "HS1_EN2"
 		(at 24.13 142.24 0)
@@
 		)
 	)
-	(label "IN3"
+	(label "IN_MCU3"
 		(at 163.83 54.61 180)
 		(effects
@@
 		)
 	)
+	(label "IN_MCU7"
+		(at 72.39 187.96 180)
+		(effects
+			(font
+				(size 1.27 1.27)
+			)
+			(justify right bottom)
+		)
+	)
 	(label "BO_IN6"
 		(at 106.68 64.77 0)
@@
 		)
 	)
-	(label "IN8"
+	(label "IN_MCU8"
 		(at 163.83 67.31 180)
 		(effects
@@
 			)
 		)
+		(pin "IN_MCU_1" input
+			(at 62.23 172.72 0)
+			(effects
+				(font
+					(size 1.27 1.27)
+				)
+				(justify right)
+			)
+		)
+		(pin "IN_MCU_2" input
+			(at 62.23 175.26 0)
+			(effects
+				(font
+					(size 1.27 1.27)
+				)
+				(justify right)
+			)
+		)
+		(pin "IN_MCU_3" input
+			(at 62.23 177.8 0)
+			(effects
+				(font
+					(size 1.27 1.27)
+				)
+				(justify right)
+			)
+		)
+		(pin "IN_MCU_4" input
+			(at 62.23 180.34 0)
+			(effects
+				(font
+					(size 1.27 1.27)
+				)
+				(justify right)
+			)
+		)
+		(pin "IN_MCU_5" input
+			(at 62.23 182.88 0)
+			(effects
+				(font
+					(size 1.27 1.27)
+				)
+				(justify right)
+			)
+		)
+		(pin "IN_MCU_6" input
+			(at 62.23 185.42 0)
+			(effects
+				(font
+					(size 1.27 1.27)
+				)
+				(justify right)
+			)
+		)
+		(pin "IN_MCU_7" input
+			(at 62.23 187.96 0)
+			(effects
+				(font
+					(size 1.27 1.27)
+				)
+				(justify right)
+			)
+		)
+		(pin "IN_MCU_8" input
+			(at 62.23 190.5 0)
+			(effects
+				(font
+					(size 1.27 1.27)
+				)
+				(justify right)
+			)
+		)
